Commit message: Update GNSS_sensor.xacro

File: urdf/GNSS_sensor.xacro (robot description, xacro)
@@ -11,5 +11,5 @@
             <origin xyz="0 0 0" rpy="0 0 0"/>
             <geometry>
-            <mesh   filename="file://$(find AMR-Sweeper_description)/meshes/Sensors/GNSS.stl" />
+            <mesh   filename="https://github.com/O-Robotics/AMR-Sweeper_description/blob/foxglove/urdf/meshes/GNSS.dae" />
             </geometry>
             <material name="black"/>

Commit message: Update GNSS_sensor.xacro

File: urdf/GNSS_sensor.xacro (robot description, xacro)
@@ -11,5 +11,5 @@
             <origin xyz="0 0 0" rpy="0 0 0"/>
             <geometry>
-            <mesh   filename="https://github.com/O-Robotics/AMR-Sweeper_description/blob/foxglove/urdf/meshes/GNSS.dae" />
+            <mesh   filename="https://raw.githubusercontent.com/O-Robotics/AMR-Sweeper_description/blob/foxglove/meshes/Sensors/GNSS.stl" />
             </geometry>
             <material name="black"/>

Commit message: Update GNSS_sensor.xacro

File: urdf/GNSS_sensor.xacro (robot description, xacro)
@@ -11,5 +11,5 @@
             <origin xyz="0 0 0" rpy="0 0 0"/>
             <geometry>
-            <mesh   filename="https://raw.githubusercontent.com/O-Robotics/AMR-Sweeper_description/blob/foxglove/meshes/Sensors/GNSS.stl" />
+            <mesh   filename="meshes/Sensors/GNSS.stl" />
             </geometry>
             <material name="black"/>

Commit message: Update GNSS_sensor.xacro

File: urdf/GNSS_sensor.xacro (robot description, xacro)
@@ -11,5 +11,5 @@
             <origin xyz="0 0 0" rpy="0 0 0"/>
             <geometry>
-            <mesh   filename="meshes/Sensors/GNSS.stl" />
+            <mesh   filename="package://amr-sweeper_description/meshes/Sensors/GNSS.stl" />
             </geometry>
             <material name="black"/>
