Commit message: Added .dae files to meshes folder within urdf

File: urdf/robot_core.xacro (robot description, xacro)
@@ -19,5 +19,5 @@
             <origin xyz="0 0 0" rpy="0 0 0"/>
             <geometry>
-                <mesh   filename="file://$(find AMR-Sweeper_description)/meshes/Chassis/Chassis.stl" />
+                <mesh   filename="file://$(find AMR-Sweeper_description)/urdf/meshes/Chassis.dae" />
             </geometry>
             <material name="grey"/>
@@ -47,5 +47,5 @@
             <origin xyz="0 0 0" rpy="${pi/2} 0 0"/>
             <geometry>
-                <mesh   filename="file://$(find AMR-Sweeper_description)/meshes/WheelAssembly/WheelAssembly.stl" />
+                <mesh   filename="file://$(find AMR-Sweeper_description)/urdf/meshes/WheelAssembly.dae" />
             </geometry>
             <material name="yellow"/>
@@ -73,5 +73,5 @@
             <origin xyz="0 0 0" rpy="${pi/2} 0 0"/>
             <geometry>
-                <mesh   filename="file://$(find AMR-Sweeper_description)/meshes/WheelAssembly/WheelAssembly.stl" />
+                <mesh   filename="file://$(find AMR-Sweeper_description)/urdf/meshes/WheelAssembly.dae" />
             </geometry>
             <material name="yellow"/>
@@ -100,5 +100,5 @@
             <origin xyz="0 0 0" rpy="0 0 0"/>
             <geometry>
-                <mesh   filename="file://$(find AMR-Sweeper_description)/meshes/Tool/Tool.stl" />
+                <mesh   filename="file://$(find AMR-Sweeper_description)/urdf/meshes/Tool.dae" />
             </geometry>
             <material name="black"/>
@@ -119,5 +119,5 @@
             <origin xyz="0 0 0" rpy="0 0 0"/>
             <geometry>
-                <mesh   filename="file://$(find AMR-Sweeper_description)/meshes/Tool/Brush.stl" />
+                <mesh   filename="file://$(find AMR-Sweeper_description)/urdf/meshes/Brush.dae" />
             </geometry>
             <material name="red"/>
@@ -144,5 +144,5 @@
             <origin xyz="0 0 0" rpy="0 0 0"/>
             <geometry>
-                <mesh   filename="file://$(find AMR-Sweeper_description)/meshes/Tool/Brush.stl" />
+                <mesh   filename="file://$(find AMR-Sweeper_description)/urdf/meshes/Tool/Brush.dae" />
             </geometry>
             <material name="red"/>

Commit message: Update robot_core.xacro

File: urdf/robot_core.xacro (robot description, xacro)
@@ -19,5 +19,5 @@
             <origin xyz="0 0 0" rpy="0 0 0"/>
             <geometry>
-                <mesh   filename="file://$(find AMR-Sweeper_description)/urdf/meshes/Chassis.dae" />
+                <mesh   filename="https://raw.githubusercontent.com/O-Robotics/AMR-Sweeper_description/blob/foxglove/urdf/meshes/Chassis.dae" />
             </geometry>
             <material name="grey"/>
@@ -27,5 +27,5 @@
             <origin xyz="0 0 0" rpy="0 0 0"/>
             <geometry>
-                <mesh   filename="file://$(find AMR-Sweeper_description)/meshes/Chassis/Chassis.stl" />
+                <mesh   filename="https://raw.githubusercontent.com/O-Robotics/AMR-Sweeper_description/blob/foxglove/meshes/Chassis/Chassis.stl" />
             </geometry>
         </collision>
@@ -47,5 +47,5 @@
             <origin xyz="0 0 0" rpy="${pi/2} 0 0"/>
             <geometry>
-                <mesh   filename="file://$(find AMR-Sweeper_description)/urdf/meshes/WheelAssembly.dae" />
+                <mesh   filename="https://raw.githubusercontent.com/O-Robotics/AMR-Sweeper_description/blob/foxglove/urdf/meshes/WheelAssembly.dae" />
             </geometry>
             <material name="yellow"/>
@@ -54,5 +54,5 @@
             <origin xyz="0 0 0" rpy="${pi/2} 0 0"/>
             <geometry>
-                <mesh   filename="file://$(find AMR-Sweeper_description)/meshes/WheelAssembly/WheelAssembly.stl" />
+                <mesh   filename="https://raw.githubusercontent.com/O-Robotics/AMR-Sweeper_description/blob/foxglove/meshes/WheelAssembly/WheelAssembly.stl" />
             </geometry>
         </collision>
@@ -73,5 +73,5 @@
             <origin xyz="0 0 0" rpy="${pi/2} 0 0"/>
             <geometry>
-                <mesh   filename="file://$(find AMR-Sweeper_description)/urdf/meshes/WheelAssembly.dae" />
+                <mesh   filename="https://raw.githubusercontent.com/O-Robotics/AMR-Sweeper_description/blob/foxglove/urdf/meshes/WheelAssembly.dae" />
             </geometry>
             <material name="yellow"/>
@@ -80,5 +80,5 @@
             <origin xyz="0 0 0" rpy="${pi/2} 0 0"/>
             <geometry>
-                <mesh   filename="file://$(find AMR-Sweeper_description)/meshes/WheelAssembly/WheelAssembly.stl" />
+                <mesh   filename="https://raw.githubusercontent.com/O-Robotics/AMR-Sweeper_description/blob/foxglove/meshes/WheelAssembly/WheelAssembly.stl" />
             </geometry>
         </collision>
@@ -100,5 +100,5 @@
             <origin xyz="0 0 0" rpy="0 0 0"/>
             <geometry>
-                <mesh   filename="file://$(find AMR-Sweeper_description)/urdf/meshes/Tool.dae" />
+                <mesh   filename="https://raw.githubusercontent.com/O-Robotics/AMR-Sweeper_description/blob/foxglove/urdf/meshes/Tool.dae" />
             </geometry>
             <material name="black"/>
@@ -119,5 +119,5 @@
             <origin xyz="0 0 0" rpy="0 0 0"/>
             <geometry>
-                <mesh   filename="file://$(find AMR-Sweeper_description)/urdf/meshes/Brush.dae" />
+                <mesh   filename="https://raw.githubusercontent.com/O-Robotics/AMR-Sweeper_description/blob/foxglove/urdf/meshes/Brush.dae" />
             </geometry>
             <material name="red"/>
@@ -126,5 +126,5 @@
             <origin xyz="0 0 0" rpy="0 0 0"/>
             <geometry>
-                <mesh   filename="file://$(find AMR-Sweeper_description)/meshes/Tool/Brush.stl" />
+                <mesh   filename="https://raw.githubusercontent.com/O-Robotics/AMR-Sweeper_description/blob/foxglove/meshes/Tool/Brush.stl" />
             </geometry>
         </collision>
@@ -144,5 +144,5 @@
             <origin xyz="0 0 0" rpy="0 0 0"/>
             <geometry>
-                <mesh   filename="file://$(find AMR-Sweeper_description)/urdf/meshes/Tool/Brush.dae" />
+                <mesh   filename="https://raw.githubusercontent.com/O-Robotics/AMR-Sweeper_description/blob/foxglove/urdf/meshes/Tool/Brush.dae" />
             </geometry>
             <material name="red"/>
@@ -151,5 +151,5 @@
             <origin xyz="0 0 0" rpy="0 0 0"/>
             <geometry>
-                <mesh   filename="file://$(find AMR-Sweeper_description)/meshes/Tool/Brush.stl" />
+                <mesh   filename="https://raw.githubusercontent.com/O-Robotics/AMR-Sweeper_description/blob/foxglove/meshes/Tool/Brush.stl" />
             </geometry>
         </collision>

Commit message: Update robot_core.xacro again

File: urdf/robot_core.xacro (robot description, xacro)
@@ -19,5 +19,5 @@
             <origin xyz="0 0 0" rpy="0 0 0"/>
             <geometry>
-                <mesh   filename="https://raw.githubusercontent.com/O-Robotics/AMR-Sweeper_description/blob/foxglove/urdf/meshes/Chassis.dae" />
+                <mesh   filename="https://github.com/O-Robotics/AMR-Sweeper_description/blob/foxglove/urdf/meshes/Chassis.dae" />
             </geometry>
             <material name="grey"/>
@@ -27,5 +27,5 @@
             <origin xyz="0 0 0" rpy="0 0 0"/>
             <geometry>
-                <mesh   filename="https://raw.githubusercontent.com/O-Robotics/AMR-Sweeper_description/blob/foxglove/meshes/Chassis/Chassis.stl" />
+                <mesh   filename="https://github.com/O-Robotics/AMR-Sweeper_description/blob/foxglove/meshes/Chassis/Chassis.stl" />
             </geometry>
         </collision>
@@ -47,5 +47,5 @@
             <origin xyz="0 0 0" rpy="${pi/2} 0 0"/>
             <geometry>
-                <mesh   filename="https://raw.githubusercontent.com/O-Robotics/AMR-Sweeper_description/blob/foxglove/urdf/meshes/WheelAssembly.dae" />
+                <mesh   filename="https://github.com/O-Robotics/AMR-Sweeper_description/blob/foxglove/urdf/meshes/WheelAssembly.dae" />
             </geometry>
             <material name="yellow"/>
@@ -54,5 +54,5 @@
             <origin xyz="0 0 0" rpy="${pi/2} 0 0"/>
             <geometry>
-                <mesh   filename="https://raw.githubusercontent.com/O-Robotics/AMR-Sweeper_description/blob/foxglove/meshes/WheelAssembly/WheelAssembly.stl" />
+                <mesh   filename="https://github.com/O-Robotics/AMR-Sweeper_description/blob/foxglove/meshes/WheelAssembly/WheelAssembly.stl" />
             </geometry>
         </collision>
@@ -73,5 +73,5 @@
             <origin xyz="0 0 0" rpy="${pi/2} 0 0"/>
             <geometry>
-                <mesh   filename="https://raw.githubusercontent.com/O-Robotics/AMR-Sweeper_description/blob/foxglove/urdf/meshes/WheelAssembly.dae" />
+                <mesh   filename="https://github.com/O-Robotics/AMR-Sweeper_description/blob/foxglove/urdf/meshes/WheelAssembly.dae" />
             </geometry>
             <material name="yellow"/>
@@ -80,5 +80,5 @@
             <origin xyz="0 0 0" rpy="${pi/2} 0 0"/>
             <geometry>
-                <mesh   filename="https://raw.githubusercontent.com/O-Robotics/AMR-Sweeper_description/blob/foxglove/meshes/WheelAssembly/WheelAssembly.stl" />
+                <mesh   filename="https://github.com/O-Robotics/AMR-Sweeper_description/blob/foxglove/meshes/WheelAssembly/WheelAssembly.stl" />
             </geometry>
         </collision>
@@ -100,5 +100,5 @@
             <origin xyz="0 0 0" rpy="0 0 0"/>
             <geometry>
-                <mesh   filename="https://raw.githubusercontent.com/O-Robotics/AMR-Sweeper_description/blob/foxglove/urdf/meshes/Tool.dae" />
+                <mesh   filename="https://github.com/O-Robotics/AMR-Sweeper_description/blob/foxglove/urdf/meshes/Tool.dae" />
             </geometry>
             <material name="black"/>
@@ -119,5 +119,5 @@
             <origin xyz="0 0 0" rpy="0 0 0"/>
             <geometry>
-                <mesh   filename="https://raw.githubusercontent.com/O-Robotics/AMR-Sweeper_description/blob/foxglove/urdf/meshes/Brush.dae" />
+                <mesh   filename="https://github.com/O-Robotics/AMR-Sweeper_description/blob/foxglove/urdf/meshes/Brush.dae" />
             </geometry>
             <material name="red"/>
@@ -126,5 +126,5 @@
             <origin xyz="0 0 0" rpy="0 0 0"/>
             <geometry>
-                <mesh   filename="https://raw.githubusercontent.com/O-Robotics/AMR-Sweeper_description/blob/foxglove/meshes/Tool/Brush.stl" />
+                <mesh   filename="https://github.com/O-Robotics/AMR-Sweeper_description/blob/foxglove/meshes/Tool/Brush.stl" />
             </geometry>
         </collision>
@@ -144,5 +144,5 @@
             <origin xyz="0 0 0" rpy="0 0 0"/>
             <geometry>
-                <mesh   filename="https://raw.githubusercontent.com/O-Robotics/AMR-Sweeper_description/blob/foxglove/urdf/meshes/Tool/Brush.dae" />
+                <mesh   filename="https://github.com/O-Robotics/AMR-Sweeper_description/blob/foxglove/urdf/meshes/Tool/Brush.dae" />
             </geometry>
             <material name="red"/>
@@ -151,5 +151,5 @@
             <origin xyz="0 0 0" rpy="0 0 0"/>
             <geometry>
-                <mesh   filename="https://raw.githubusercontent.com/O-Robotics/AMR-Sweeper_description/blob/foxglove/meshes/Tool/Brush.stl" />
+                <mesh   filename="https://github.com/O-Robotics/AMR-Sweeper_description/blob/foxglove/meshes/Tool/Brush.stl" />
             </geometry>
         </collision>

Commit message: Update robot_core.xacro

File: urdf/robot_core.xacro (robot description, xacro)
@@ -19,5 +19,5 @@
             <origin xyz="0 0 0" rpy="0 0 0"/>
             <geometry>
-                <mesh   filename="https://github.com/O-Robotics/AMR-Sweeper_description/blob/foxglove/urdf/meshes/Chassis.dae" />
+                <mesh   filename="https://raw.githubusercontent.com/O-Robotics/AMR-Sweeper_description/blob/foxglove/meshes/Chassis/Chassis.stl" />
             </geometry>
             <material name="grey"/>
@@ -27,5 +27,5 @@
             <origin xyz="0 0 0" rpy="0 0 0"/>
             <geometry>
-                <mesh   filename="https://github.com/O-Robotics/AMR-Sweeper_description/blob/foxglove/meshes/Chassis/Chassis.stl" />
+                <mesh   filename="https://raw.githubusercontent.com/O-Robotics/AMR-Sweeper_description/blob/foxglove/meshes/Chassis/Chassis.stl" />
             </geometry>
         </collision>
@@ -47,5 +47,5 @@
             <origin xyz="0 0 0" rpy="${pi/2} 0 0"/>
             <geometry>
-                <mesh   filename="https://github.com/O-Robotics/AMR-Sweeper_description/blob/foxglove/urdf/meshes/WheelAssembly.dae" />
+                <mesh   filename="https://raw.githubusercontent.com/O-Robotics/AMR-Sweeper_description/blob/foxglove/meshes/WheelAssembly/WheelAssembly.stl" />
             </geometry>
             <material name="yellow"/>
@@ -54,5 +54,5 @@
             <origin xyz="0 0 0" rpy="${pi/2} 0 0"/>
             <geometry>
-                <mesh   filename="https://github.com/O-Robotics/AMR-Sweeper_description/blob/foxglove/meshes/WheelAssembly/WheelAssembly.stl" />
+                <mesh   filename="https://raw.githubusercontent.com/O-Robotics/AMR-Sweeper_description/blob/foxglove/meshes/WheelAssembly/WheelAssembly.stl" />
             </geometry>
         </collision>
@@ -73,5 +73,5 @@
             <origin xyz="0 0 0" rpy="${pi/2} 0 0"/>
             <geometry>
-                <mesh   filename="https://github.com/O-Robotics/AMR-Sweeper_description/blob/foxglove/urdf/meshes/WheelAssembly.dae" />
+                <mesh   filename="https://raw.githubusercontent.com/O-Robotics/AMR-Sweeper_description/blob/foxglove/meshes/WheelAssembly/WheelAssembly.stl" />
             </geometry>
             <material name="yellow"/>
@@ -80,5 +80,5 @@
             <origin xyz="0 0 0" rpy="${pi/2} 0 0"/>
             <geometry>
-                <mesh   filename="https://github.com/O-Robotics/AMR-Sweeper_description/blob/foxglove/meshes/WheelAssembly/WheelAssembly.stl" />
+                <mesh   filename="https://raw.githubusercontent.com/O-Robotics/AMR-Sweeper_description/blob/foxglove/meshes/WheelAssembly/WheelAssembly.stl" />
             </geometry>
         </collision>
@@ -100,5 +100,5 @@
             <origin xyz="0 0 0" rpy="0 0 0"/>
             <geometry>
-                <mesh   filename="https://github.com/O-Robotics/AMR-Sweeper_description/blob/foxglove/urdf/meshes/Tool.dae" />
+                <mesh   filename="https://raw.githubusercontent.com/O-Robotics/AMR-Sweeper_description/blob/foxglove/meshes/Tool/Tool.stl" />
             </geometry>
             <material name="black"/>
@@ -119,5 +119,5 @@
             <origin xyz="0 0 0" rpy="0 0 0"/>
             <geometry>
-                <mesh   filename="https://github.com/O-Robotics/AMR-Sweeper_description/blob/foxglove/urdf/meshes/Brush.dae" />
+                <mesh   filename="https://raw.githubusercontent.com/O-Robotics/AMR-Sweeper_description/blob/foxglove/meshes/Tool/Brush.stl" />
             </geometry>
             <material name="red"/>
@@ -126,5 +126,5 @@
             <origin xyz="0 0 0" rpy="0 0 0"/>
             <geometry>
-                <mesh   filename="https://github.com/O-Robotics/AMR-Sweeper_description/blob/foxglove/meshes/Tool/Brush.stl" />
+                <mesh   filename="https://raw.githubusercontent.com/O-Robotics/AMR-Sweeper_description/blob/foxglove/meshes/Tool/Brush.stl" />
             </geometry>
         </collision>
@@ -144,5 +144,5 @@
             <origin xyz="0 0 0" rpy="0 0 0"/>
             <geometry>
-                <mesh   filename="https://github.com/O-Robotics/AMR-Sweeper_description/blob/foxglove/urdf/meshes/Tool/Brush.dae" />
+                <mesh   filename="https://raw.githubusercontent.com/O-Robotics/AMR-Sweeper_description/blob/foxglove/meshes/Tool/Brush.stl" />
             </geometry>
             <material name="red"/>
@@ -151,5 +151,5 @@
             <origin xyz="0 0 0" rpy="0 0 0"/>
             <geometry>
-                <mesh   filename="https://github.com/O-Robotics/AMR-Sweeper_description/blob/foxglove/meshes/Tool/Brush.stl" />
+                <mesh   filename="https://raw.githubusercontent.com/O-Robotics/AMR-Sweeper_description/blob/foxglove/meshes/Tool/Brush.stl" />
             </geometry>
         </collision>

Commit message: Update robot_core.xacro

File: urdf/robot_core.xacro (robot description, xacro)
@@ -19,5 +19,5 @@
             <origin xyz="0 0 0" rpy="0 0 0"/>
             <geometry>
-                <mesh   filename="https://raw.githubusercontent.com/O-Robotics/AMR-Sweeper_description/blob/foxglove/meshes/Chassis/Chassis.stl" />
+                <mesh   filename="meshes/Chassis/Chassis.stl" />
             </geometry>
             <material name="grey"/>
@@ -27,5 +27,5 @@
             <origin xyz="0 0 0" rpy="0 0 0"/>
             <geometry>
-                <mesh   filename="https://raw.githubusercontent.com/O-Robotics/AMR-Sweeper_description/blob/foxglove/meshes/Chassis/Chassis.stl" />
+                <mesh   filename="meshes/Chassis/Chassis.stl" />
             </geometry>
         </collision>
@@ -47,5 +47,5 @@
             <origin xyz="0 0 0" rpy="${pi/2} 0 0"/>
             <geometry>
-                <mesh   filename="https://raw.githubusercontent.com/O-Robotics/AMR-Sweeper_description/blob/foxglove/meshes/WheelAssembly/WheelAssembly.stl" />
+                <mesh   filename="meshes/WheelAssembly/WheelAssembly.stl" />
             </geometry>
             <material name="yellow"/>
@@ -54,5 +54,5 @@
             <origin xyz="0 0 0" rpy="${pi/2} 0 0"/>
             <geometry>
-                <mesh   filename="https://raw.githubusercontent.com/O-Robotics/AMR-Sweeper_description/blob/foxglove/meshes/WheelAssembly/WheelAssembly.stl" />
+                <mesh   filename="meshes/WheelAssembly/WheelAssembly.stl" />
             </geometry>
         </collision>
@@ -73,5 +73,5 @@
             <origin xyz="0 0 0" rpy="${pi/2} 0 0"/>
             <geometry>
-                <mesh   filename="https://raw.githubusercontent.com/O-Robotics/AMR-Sweeper_description/blob/foxglove/meshes/WheelAssembly/WheelAssembly.stl" />
+                <mesh   filename="meshes/WheelAssembly/WheelAssembly.stl" />
             </geometry>
             <material name="yellow"/>
@@ -80,5 +80,5 @@
             <origin xyz="0 0 0" rpy="${pi/2} 0 0"/>
             <geometry>
-                <mesh   filename="https://raw.githubusercontent.com/O-Robotics/AMR-Sweeper_description/blob/foxglove/meshes/WheelAssembly/WheelAssembly.stl" />
+                <mesh   filename="meshes/WheelAssembly/WheelAssembly.stl" />
             </geometry>
         </collision>
@@ -100,5 +100,5 @@
             <origin xyz="0 0 0" rpy="0 0 0"/>
             <geometry>
-                <mesh   filename="https://raw.githubusercontent.com/O-Robotics/AMR-Sweeper_description/blob/foxglove/meshes/Tool/Tool.stl" />
+                <mesh   filename="meshes/Tool/Tool.stl" />
             </geometry>
             <material name="black"/>
@@ -119,5 +119,5 @@
             <origin xyz="0 0 0" rpy="0 0 0"/>
             <geometry>
-                <mesh   filename="https://raw.githubusercontent.com/O-Robotics/AMR-Sweeper_description/blob/foxglove/meshes/Tool/Brush.stl" />
+                <mesh   filename="meshes/Tool/Brush.stl" />
             </geometry>
             <material name="red"/>
@@ -126,5 +126,5 @@
             <origin xyz="0 0 0" rpy="0 0 0"/>
             <geometry>
-                <mesh   filename="https://raw.githubusercontent.com/O-Robotics/AMR-Sweeper_description/blob/foxglove/meshes/Tool/Brush.stl" />
+                <mesh   filename="meshes/Tool/Brush.stl" />
             </geometry>
         </collision>
@@ -144,5 +144,5 @@
             <origin xyz="0 0 0" rpy="0 0 0"/>
             <geometry>
-                <mesh   filename="https://raw.githubusercontent.com/O-Robotics/AMR-Sweeper_description/blob/foxglove/meshes/Tool/Brush.stl" />
+                <mesh   filename="meshes/Tool/Brush.stl" />
             </geometry>
             <material name="red"/>
@@ -151,5 +151,5 @@
             <origin xyz="0 0 0" rpy="0 0 0"/>
             <geometry>
-                <mesh   filename="https://raw.githubusercontent.com/O-Robotics/AMR-Sweeper_description/blob/foxglove/meshes/Tool/Brush.stl" />
+                <mesh   filename="meshes/Tool/Brush.stl" />
             </geometry>
         </collision>
