Commit message: Update robot_core.xacro
added package://AMR-Sweeper_description/ to filename

File: urdf/robot_core.xacro (robot description, xacro)
@@ -19,5 +19,5 @@
             <origin xyz="0 0 0" rpy="0 0 0"/>
             <geometry>
-                <mesh   filename="meshes/Chassis/Chassis.stl" />
+                <mesh   filename="package://AMR-Sweeper_description/meshes/Chassis/Chassis.stl" />
             </geometry>
             <material name="grey"/>
@@ -27,5 +27,5 @@
             <origin xyz="0 0 0" rpy="0 0 0"/>
             <geometry>
-                <mesh   filename="meshes/Chassis/Chassis.stl" />
+                <mesh   filename="package://AMR-Sweeper_description/meshes/Chassis/Chassis.stl" />
             </geometry>
         </collision>
@@ -47,5 +47,5 @@
             <origin xyz="0 0 0" rpy="${pi/2} 0 0"/>
             <geometry>
-                <mesh   filename="meshes/WheelAssembly/WheelAssembly.stl" />
+                <mesh   filename="package://AMR-Sweeper_description/meshes/WheelAssembly/WheelAssembly.stl" />
             </geometry>
             <material name="yellow"/>
@@ -54,5 +54,5 @@
             <origin xyz="0 0 0" rpy="${pi/2} 0 0"/>
             <geometry>
-                <mesh   filename="meshes/WheelAssembly/WheelAssembly.stl" />
+                <mesh   filename="package://AMR-Sweeper_description/meshes/WheelAssembly/WheelAssembly.stl" />
             </geometry>
         </collision>
@@ -73,5 +73,5 @@
             <origin xyz="0 0 0" rpy="${pi/2} 0 0"/>
             <geometry>
-                <mesh   filename="meshes/WheelAssembly/WheelAssembly.stl" />
+                <mesh   filename="package://AMR-Sweeper_description/meshes/WheelAssembly/WheelAssembly.stl" />
             </geometry>
             <material name="yellow"/>
@@ -80,5 +80,5 @@
             <origin xyz="0 0 0" rpy="${pi/2} 0 0"/>
             <geometry>
-                <mesh   filename="meshes/WheelAssembly/WheelAssembly.stl" />
+                <mesh   filename="package://AMR-Sweeper_description/meshes/WheelAssembly/WheelAssembly.stl" />
             </geometry>
         </collision>
@@ -100,5 +100,5 @@
             <origin xyz="0 0 0" rpy="0 0 0"/>
             <geometry>
-                <mesh   filename="meshes/Tool/Tool.stl" />
+                <mesh   filename="package://AMR-Sweeper_description/meshes/Tool/Tool.stl" />
             </geometry>
             <material name="black"/>
@@ -119,5 +119,5 @@
             <origin xyz="0 0 0" rpy="0 0 0"/>
             <geometry>
-                <mesh   filename="meshes/Tool/Brush.stl" />
+                <mesh   filename="package://AMR-Sweeper_description/meshes/Tool/Brush.stl" />
             </geometry>
             <material name="red"/>
@@ -126,5 +126,5 @@
             <origin xyz="0 0 0" rpy="0 0 0"/>
             <geometry>
-                <mesh   filename="meshes/Tool/Brush.stl" />
+                <mesh   filename="package://AMR-Sweeper_description/meshes/Tool/Brush.stl" />
             </geometry>
         </collision>
@@ -144,5 +144,5 @@
             <origin xyz="0 0 0" rpy="0 0 0"/>
             <geometry>
-                <mesh   filename="meshes/Tool/Brush.stl" />
+                <mesh   filename="package://AMR-Sweeper_description/meshes/Tool/Brush.stl" />
             </geometry>
             <material name="red"/>
@@ -151,5 +151,5 @@
             <origin xyz="0 0 0" rpy="0 0 0"/>
             <geometry>
-                <mesh   filename="meshes/Tool/Brush.stl" />
+                <mesh   filename="package://AMR-Sweeper_description/meshes/Tool/Brush.stl" />
             </geometry>
         </collision>

Commit message: Update robot_core.xacro

File: urdf/robot_core.xacro (robot description, xacro)
@@ -19,5 +19,5 @@
             <origin xyz="0 0 0" rpy="0 0 0"/>
             <geometry>
-                <mesh   filename="package://AMR-Sweeper_description/meshes/Chassis/Chassis.stl" />
+                <mesh   filename="package://amr-sweeper_description/meshes/Chassis/Chassis.stl" />
             </geometry>
             <material name="grey"/>
@@ -27,5 +27,5 @@
             <origin xyz="0 0 0" rpy="0 0 0"/>
             <geometry>
-                <mesh   filename="package://AMR-Sweeper_description/meshes/Chassis/Chassis.stl" />
+                <mesh   filename="package://amr-sweeper_description/meshes/Chassis/Chassis.stl" />
             </geometry>
         </collision>
@@ -47,5 +47,5 @@
             <origin xyz="0 0 0" rpy="${pi/2} 0 0"/>
             <geometry>
-                <mesh   filename="package://AMR-Sweeper_description/meshes/WheelAssembly/WheelAssembly.stl" />
+                <mesh   filename="package://amr-sweeper_description/meshes/WheelAssembly/WheelAssembly.stl" />
             </geometry>
             <material name="yellow"/>
@@ -54,5 +54,5 @@
             <origin xyz="0 0 0" rpy="${pi/2} 0 0"/>
             <geometry>
-                <mesh   filename="package://AMR-Sweeper_description/meshes/WheelAssembly/WheelAssembly.stl" />
+                <mesh   filename="package://amr-sweeper_description/meshes/WheelAssembly/WheelAssembly.stl" />
             </geometry>
         </collision>
@@ -73,5 +73,5 @@
             <origin xyz="0 0 0" rpy="${pi/2} 0 0"/>
             <geometry>
-                <mesh   filename="package://AMR-Sweeper_description/meshes/WheelAssembly/WheelAssembly.stl" />
+                <mesh   filename="package://amr-sweeper_description/meshes/WheelAssembly/WheelAssembly.stl" />
             </geometry>
             <material name="yellow"/>
@@ -80,5 +80,5 @@
             <origin xyz="0 0 0" rpy="${pi/2} 0 0"/>
             <geometry>
-                <mesh   filename="package://AMR-Sweeper_description/meshes/WheelAssembly/WheelAssembly.stl" />
+                <mesh   filename="package://amr-sweeper_description/meshes/WheelAssembly/WheelAssembly.stl" />
             </geometry>
         </collision>
@@ -100,5 +100,5 @@
             <origin xyz="0 0 0" rpy="0 0 0"/>
             <geometry>
-                <mesh   filename="package://AMR-Sweeper_description/meshes/Tool/Tool.stl" />
+                <mesh   filename="package://amr-sweeper_description/meshes/Tool/Tool.stl" />
             </geometry>
             <material name="black"/>
@@ -119,5 +119,5 @@
             <origin xyz="0 0 0" rpy="0 0 0"/>
             <geometry>
-                <mesh   filename="package://AMR-Sweeper_description/meshes/Tool/Brush.stl" />
+                <mesh   filename="package://amr-sweeper_description/meshes/Tool/Brush.stl" />
             </geometry>
             <material name="red"/>
@@ -126,5 +126,5 @@
             <origin xyz="0 0 0" rpy="0 0 0"/>
             <geometry>
-                <mesh   filename="package://AMR-Sweeper_description/meshes/Tool/Brush.stl" />
+                <mesh   filename="package://amr-sweeper_description/meshes/Tool/Brush.stl" />
             </geometry>
         </collision>
@@ -144,5 +144,5 @@
             <origin xyz="0 0 0" rpy="0 0 0"/>
             <geometry>
-                <mesh   filename="package://AMR-Sweeper_description/meshes/Tool/Brush.stl" />
+                <mesh   filename="package://amr-sweeper_description/meshes/Tool/Brush.stl" />
             </geometry>
             <material name="red"/>
@@ -151,5 +151,5 @@
             <origin xyz="0 0 0" rpy="0 0 0"/>
             <geometry>
-                <mesh   filename="package://AMR-Sweeper_description/meshes/Tool/Brush.stl" />
+                <mesh   filename="package://amr-sweeper_description/meshes/Tool/Brush.stl" />
             </geometry>
         </collision>

Commit message: Update robot_core.xacro

File: urdf/robot_core.xacro (robot description, xacro)
@@ -19,5 +19,5 @@
             <origin xyz="0 0 0" rpy="0 0 0"/>
             <geometry>
-                <mesh   filename="package://amr-sweeper_description/meshes/Chassis/Chassis.stl" />
+                <mesh   filename="package://amrsweeper_description/meshes/Chassis/Chassis.stl" />
             </geometry>
             <material name="grey"/>
@@ -27,5 +27,5 @@
             <origin xyz="0 0 0" rpy="0 0 0"/>
             <geometry>
-                <mesh   filename="package://amr-sweeper_description/meshes/Chassis/Chassis.stl" />
+                <mesh   filename="package://amrsweeper_description/meshes/Chassis/Chassis.stl" />
             </geometry>
         </collision>
@@ -47,5 +47,5 @@
             <origin xyz="0 0 0" rpy="${pi/2} 0 0"/>
             <geometry>
-                <mesh   filename="package://amr-sweeper_description/meshes/WheelAssembly/WheelAssembly.stl" />
+                <mesh   filename="package://amrsweeper_description/meshes/WheelAssembly/WheelAssembly.stl" />
             </geometry>
             <material name="yellow"/>
@@ -54,5 +54,5 @@
             <origin xyz="0 0 0" rpy="${pi/2} 0 0"/>
             <geometry>
-                <mesh   filename="package://amr-sweeper_description/meshes/WheelAssembly/WheelAssembly.stl" />
+                <mesh   filename="package://amrsweeper_description/meshes/WheelAssembly/WheelAssembly.stl" />
             </geometry>
         </collision>
@@ -73,5 +73,5 @@
             <origin xyz="0 0 0" rpy="${pi/2} 0 0"/>
             <geometry>
-                <mesh   filename="package://amr-sweeper_description/meshes/WheelAssembly/WheelAssembly.stl" />
+                <mesh   filename="package://amrsweeper_description/meshes/WheelAssembly/WheelAssembly.stl" />
             </geometry>
             <material name="yellow"/>
@@ -80,5 +80,5 @@
             <origin xyz="0 0 0" rpy="${pi/2} 0 0"/>
             <geometry>
-                <mesh   filename="package://amr-sweeper_description/meshes/WheelAssembly/WheelAssembly.stl" />
+                <mesh   filename="package://amrsweeper_description/meshes/WheelAssembly/WheelAssembly.stl" />
             </geometry>
         </collision>
@@ -100,5 +100,5 @@
             <origin xyz="0 0 0" rpy="0 0 0"/>
             <geometry>
-                <mesh   filename="package://amr-sweeper_description/meshes/Tool/Tool.stl" />
+                <mesh   filename="package://amrsweeper_description/meshes/Tool/Tool.stl" />
             </geometry>
             <material name="black"/>
@@ -119,5 +119,5 @@
             <origin xyz="0 0 0" rpy="0 0 0"/>
             <geometry>
-                <mesh   filename="package://amr-sweeper_description/meshes/Tool/Brush.stl" />
+                <mesh   filename="package://amrsweeper_description/meshes/Tool/Brush.stl" />
             </geometry>
             <material name="red"/>
@@ -126,5 +126,5 @@
             <origin xyz="0 0 0" rpy="0 0 0"/>
             <geometry>
-                <mesh   filename="package://amr-sweeper_description/meshes/Tool/Brush.stl" />
+                <mesh   filename="package://amrsweeper_description/meshes/Tool/Brush.stl" />
             </geometry>
         </collision>
@@ -144,5 +144,5 @@
             <origin xyz="0 0 0" rpy="0 0 0"/>
             <geometry>
-                <mesh   filename="package://amr-sweeper_description/meshes/Tool/Brush.stl" />
+                <mesh   filename="package://amrsweeper_description/meshes/Tool/Brush.stl" />
             </geometry>
             <material name="red"/>
@@ -151,5 +151,5 @@
             <origin xyz="0 0 0" rpy="0 0 0"/>
             <geometry>
-                <mesh   filename="package://amr-sweeper_description/meshes/Tool/Brush.stl" />
+                <mesh   filename="package://amrsweeper_description/meshes/Tool/Brush.stl" />
             </geometry>
         </collision>
